Commit message: Add gripper embodiment + palm-depth diagnostic
- New NERO + parallel-jaw gripper embodiment alongside inspire hand:
  nero_gripper_right.urdf (arm chain + 2 prismatic fingers), specs
  NERO_GRIPPER_RGB/RGBD in robot_specs.py, viz_urdf field.
- derive_embodiment.py: branch on hand_mode; gripper via thumb-index
  pinch distance -> gripper width; dynamic state dim (8 gripper / 13 inspire).
- replay_rerun.py: expand gripper_joint -> both finger joints; load viz_urdf.
- Web: embodiment selector is now a dropdown (inspire / gripper), hand param
  threaded through app_web.py pipeline.
- measure_palm_depth.py: one-shot diagnostic. On kinect2 data, palm knuckle
  depth is 100% valid, 1.4mm plane residual; depth vs monocular wrist normal
  disagrees 18.6 deg median -> motivates depth-fit wrist orientation.
- stand_v2.urdf: package:// -> relative mesh paths (loads without ROS).

File: assets/nero_description/urdf/nero_description_stand_v2.urdf (robot description, URDF)
Before this commit: robot nero_description, 10 links, 9 joints
Links:
- link base_link: geometry collision mesh filename=../../assets/nero_description/meshes/base_link.STL; visual mesh filename=../../assets/nero_description/meshes/dae/base_link.dae
- link end_effector: geometry collision mesh filename=../../assets/nero_description/meshes/stand_v2.dae; visual mesh filename=../../assets/nero_description/meshes/stand_v2.dae
- link link1: geometry collision mesh filename=../../assets/nero_description/meshes/Link1.STL; visual mesh filename=../../assets/nero_description/meshes/dae/link1.dae
- link link2: geometry collision mesh filename=../../assets/nero_description/meshes/Link2.STL; visual mesh filename=../../assets/nero_description/meshes/dae/link2.dae
- link link3: geometry collision mesh filename=../../assets/nero_description/meshes/Link3.STL; visual mesh filename=../../assets/nero_description/meshes/dae/link3.dae
- link link4: geometry collision mesh filename=../../assets/nero_description/meshes/Link4.STL; visual mesh filename=../../assets/nero_description/meshes/dae/link4.dae
- link link5: geometry collision mesh filename=../../assets/nero_description/meshes/Link5.STL; visual mesh filename=../../assets/nero_description/meshes/dae/link5.dae
- link link6: geometry collision mesh filename=../../assets/nero_description/meshes/Link6.STL; visual mesh filename=../../assets/nero_description/meshes/dae/link6.dae
- link link7: geometry collision mesh filename=../../assets/nero_description/meshes/Link7.STL; visual mesh filename=../../assets/nero_description/meshes/dae/link7.dae
