Commit message: docs: 创建结构化文档系统 + 临时修复hand_pinch/hand_ok
新增文档:
- HANDBOOK.md: 开发手册（项目结构、代码说明、开发流程）
- HARDWARE.md: 硬件文档（规格、协议、故障排除）
- CHANGELOG.md: 更新日志（整合自更新日志.md）
- PROJECT_STATUS.md: 项目进度（整合progress.md + PROJECT_PLAN.md）
- README_DOCS.md: 文档导航
- DOC_SUMMARY.md: 文档整理总结
- ASSEMBLY_SUCCESS.md/WEB_COMBO_UPDATE.md: 装配和Web更新记录

修复:
- sim/skills/gestures.yaml: hand_ok的index从limit改为0.24
- sim/skills/registry.yaml: hand_pinch的index从limit改为0.24
  (临时绕过T=141时的假阳性检查，待t6实测后改回limit)

其他:
- 更新装配URDF和combo可视化配置
- 新增combo迁移脚本

File: assets/assembled/nero_inspire_right.urdf (robot description, URDF)
Before this commit: robot nero_inspire_right, 24 links, 23 joints
Joints:
- joint flange_to_hand: origin xyz=0.000042 0.005962 0.002158 rpy=0 0 1.570796 -> xyz=0.000042 0. 0.002158 rpy=0 0 1.570796

File: assets/viz/combo/nero_inspire_right_viz.urdf (robot description, URDF)
Before this commit: robot nero_inspire_right, 30 links, 29 joints
Links:
- removed link base
- removed link hand_base_link
- removed link index_intermediate
- removed link index_proximal
- removed link index_tip
- removed link middle_intermediate
- removed link middle_proximal
- removed link middle_tip
- removed link pinky_intermediate
- removed link pinky_proximal
- removed link pinky_tip
- removed link ring_intermediate
- removed link ring_proximal
- removed link ring_tip
- removed link thumb_distal
- removed link thumb_intermediate
- removed link thumb_proximal
- removed link thumb_proximal_base
- removed link thumb_tip
- added link R_base_link, mass 0.38756; visual mesh filename=meshes/R_base_link.glb
- added link right_index_1, mass 0.01229; visual mesh filename=meshes/right_index_1.glb
- added link right_index_2, mass 0.00633; visual mesh filename=meshes/right_index_2.glb
- added link right_little_1, mass 0.012289999999999999; visual mesh filename=meshes/right_little_1.glb
- added link right_little_2, mass 0.00525; visual mesh filename=meshes/right_little_2.glb
- added link right_middle_1, mass 0.01229; visual mesh filename=meshes/right_middle_1.glb
- added link right_middle_2, mass 0.00681; visual mesh filename=meshes/right_middle_2.glb
- added link right_ring_1, mass 0.01229; visual mesh filename=meshes/right_ring_1.glb
- added link right_ring_2, mass 0.00633; visual mesh filename=meshes/right_ring_2.glb
- added link right_thumb_1, mass 0.00483; visual mesh filename=meshes/right_thumb_1.glb
- added link right_thumb_2, mass 0.05759; visual mesh filename=meshes/right_thumb_2.glb
- added link right_thumb_3, mass 0.00985; visual mesh filename=meshes/right_thumb_3.glb
- added link right_thumb_4, mass 0.00552; visual mesh filename=meshes/right_thumb_4.glb
Joints:
- removed joint base_joint
- removed joint index_intermediate_joint
- removed joint index_proximal_joint
- removed joint index_tip_joint
- removed joint middle_intermediate_joint
- removed joint middle_proximal_joint
- removed joint middle_tip_joint
- removed joint pinky_intermediate_joint
- removed joint pinky_proximal_joint
- removed joint pinky_tip_joint
- removed joint ring_intermediate_joint
- removed joint ring_proximal_joint
- removed joint ring_tip_joint
- removed joint thumb_distal_joint
- removed joint thumb_intermediate_joint
- removed joint thumb_proximal_pitch_joint
- removed joint thumb_proximal_yaw_joint
- removed joint thumb_tip_joint
- added joint right_index_1_joint: type revolute, parent R_base_link, child right_index_1, origin xyz=-0.000285333323388565 0.0202750317161709 0.136945958498439 rpy=1.53588974175501 0 0, axis 0 -0.0697564737441209 -0.997564050259825, limit lower=0 upper=1.333 effort=50 velocity=1
- added joint right_index_2_joint: type revolute, parent right_index_1, child right_index_2, origin xyz=0.0080992697963248 0.0310949249595195 -0.001 rpy=0 0 0, axis 0 0 -1, limit lower=0 upper=1.527 effort=50 velocity=1, mimic joint=right_index_1_joint multiplier=1.1169 offset=0
- added joint right_little_1_joint: type revolute, parent R_base_link, child right_little_1, origin xyz=-0.000285333323391146 -0.0374222941312603 0.134460099927073 rpy=1.67551608191454 0 0, axis 0 0 -1, limit lower=0 upper=1.333 effort=50 velocity=1
- added joint right_little_2_joint: type revolute, parent right_little_1, child right_little_2, origin xyz=0.0080966 0.031096 -0.001 rpy=0 0 0, axis 0 0 -1, limit lower=0 upper=1.527 effort=50 velocity=1, mimic joint=right_little_1_joint multiplier=1.1169 offset=0
- added joint right_middle_1_joint: type revolute, parent R_base_link, child right_middle_1, origin xyz=-0.000285333314556269 0.00295000000023597 0.137100000000016 rpy=1.5707963267792 0 0, axis 0 0 -1, limit lower=0 upper=1.333 effort=50 velocity=1
- added joint right_middle_2_joint: type revolute, parent right_middle_1, child right_middle_2, origin xyz=0.00809959893697584 0.0310948392266618 0.00100000000000044 rpy=0 0 0, axis 0 0 -1, limit lower=0 upper=1.527 effort=50 velocity=1, mimic joint=right_middle_1_joint multiplier=1.1169 offset=0
- added joint right_ring_1_joint: type revolute, parent R_base_link, child right_ring_1, origin xyz=-0.000285333323395365 -0.0182707111726564 0.136282456905841 rpy=1.62315620435472 0 0, axis 0 0 -1, limit lower=0 upper=1.333 effort=50 velocity=1
- added joint right_ring_2_joint: type revolute, parent right_ring_1, child right_ring_2, origin xyz=0.00809885846186154 0.0310950320965672 -0.001 rpy=0 0 0, axis 0 0 -1, limit lower=0 upper=1.527 effort=50 velocity=1, mimic joint=right_ring_1_joint multiplier=1.1169 offset=0
- added joint right_thumb_1_joint: type revolute, parent R_base_link, child right_thumb_1, origin xyz=0.0169600000000007 0.020450000002209 0.0663500000000002 rpy=0 0 0, axis 0 0 -1, limit lower=0 upper=1.246165 effort=50 velocity=1
- added joint right_thumb_2_joint: type revolute, parent right_thumb_1, child right_thumb_2, origin xyz=0.0107353075101483 0.00900017625730479 -0.00649999999999998 rpy=1.57079632679489 0 1.30550628049177, axis 0 0 1, limit lower=0 upper=0.48 effort=50 velocity=1
- added joint right_thumb_3_joint: type revolute, parent right_thumb_2, child right_thumb_3, origin xyz=0.0376167925538582 0.0414855421501229 -0.000800000000000356 rpy=0 0 0, axis 0 0 1, limit lower=0 upper=0.3578 effort=50 velocity=1, mimic joint=right_thumb_2_joint multiplier=1.1425 offset=0
- added joint right_thumb_4_joint: type revolute, parent right_thumb_3, child right_thumb_4, origin xyz=0.0149571022375899 0.0170124132550165 -0.00120000000000001 rpy=0 0 0, axis 0 0 1, limit lower=0 upper=0.2775 effort=50 velocity=1, mimic joint=right_thumb_3_joint multiplier=0.7508 offset=0
- joint flange_to_hand: child base -> R_base_link; origin xyz=0.000042 0.005962 0.002158 rpy=0 0 1.570796 -> xyz=0.000042 0. 0.002158 rpy=0 0 1.570796
