Commit message: fix(web): improve live hand tracking response

File: assets/hand/urdf/inspire_hand_right_6dof.urdf (robot description, URDF)
Before this commit: robot urdf_right_2025_4_18, 13 links, 12 joints
Links:
- added link index_tip
- added link middle_tip
- added link pinky_tip
- added link ring_tip
- added link thumb_tip
Joints:
- added joint index_tip_joint: type fixed, parent right_index_2, child index_tip, origin xyz=0.0144754 0.0426952 -0.0056212 rpy=0 0 0
- added joint middle_tip_joint: type fixed, parent right_middle_2, child middle_tip, origin xyz=0.0161153 0.0456677 -0.0060162 rpy=0 0 0
- added joint pinky_tip_joint: type fixed, parent right_little_2, child pinky_tip, origin xyz=0.0117575 0.0353353 -0.0059712 rpy=0 0 0
- added joint ring_tip_joint: type fixed, parent right_ring_2, child ring_tip, origin xyz=0.0144739 0.0426943 -0.0056256 rpy=0 0 0
- added joint thumb_tip_joint: type fixed, parent right_thumb_4, child thumb_tip, origin xyz=0.0137599 0.0204399 -0.0080762 rpy=0 0 0
